Commit message: Changed all references to world frame to work with Gazebo sim, incresed max speed in state machine

File: src/robot_bringup/urdf/robot.urdf (robot description, URDF)
Before this commit: robot simple_robot, 3 links, 2 joints
Links:
- removed link odom
- added link world
Joints:
- removed joint odom_to_base
- added joint world_to_base: type fixed, parent world, child base_link, origin xyz=0 0 0 rpy=0 0 0
